Commit message: 分离nav2的tf发布信息，融合手柄控制节点

File: src/px4_ego_py/urdf/px4_frame_links.urdf (robot description, URDF)
Before this commit: robot px4_frame_links, 5 links, 4 joints
Joints:
- removed joint base_link_to_base_footprint
- added joint base_link_to_base_link: type fixed, parent base_footprint, child base_link, origin xyz=0 0 0 rpy=0 0 0

Commit message: 交给gemini测试

File: src/px4_ego_py/urdf/px4_frame_links.urdf (robot description, URDF)
Before this commit: robot px4_frame_links, 5 links, 4 joints
Links:
- removed link link
- added link imu_link
Joints:
- removed joint base_link_to_base_link
- removed joint base_link_to_link
- added joint base_footprint_to_base_link: type fixed, parent base_footprint, child base_link, origin xyz=0 0 0 rpy=0 0 0
- added joint base_link_to_imu_link: type fixed, parent base_link, child imu_link, origin xyz=0 0 0 rpy=0 0 0
